Commit message: Update dami2.urdf.xacro

File: dami2_description/urdf/dami2.urdf.xacro (robot description, xacro)
@@ -160,5 +160,5 @@
   <joint name="scan_joint" type="fixed">
     <parent link="base_link"/>
-    <child link="base_scan"/>
+    <child link="camer_scan"/>
     <origin xyz="-0.054025 0.0 0.14405" rpy="0 0 0"/>
   </joint>
