Commit message: model edit1

File: dami2_description/urdf/dami2.gazebo.xacro (robot description, xacro)
@@ -101,5 +101,5 @@
     </plugin>
   </gazebo>
-  <gazebo reference="base_scan">
+  <gazebo reference="camera_link">
     <material>Gazebo/FlatBlack</material>
     <sensor type="ray" name="lds_lfcd_sensor">

File: dami2_description/urdf/dami2.urdf.xacro (robot description, xacro)
@@ -14,5 +14,5 @@
       <origin xyz="0.0 0.0 0.0" rpy="0 0 0"/>
       <geometry>
-        <mesh filename="package://dami2_description/meshes/bases/dami2_base.stl" scale="0.001 0.001 0.001"/>
+        <mesh filename="package://dami2_description/meshes/bases/base_rev.stl" scale="0.001 0.001 0.001"/>
       </geometry>
       <material name="light_black"/>
@@ -147,5 +147,5 @@
     <parent link="base_link"/>
     <child link="imu_link"/>
-    <origin xyz="0.0 0.0 0.0705" rpy="0 0 0"/>
+    <origin xyz="0.0 0.0 0.0805" rpy="0 0 0"/>
   </joint>
   <link name="imu_link">
@@ -160,6 +160,6 @@
   <joint name="scan_joint" type="fixed">
     <parent link="base_link"/>
-    <child link="base_scan"/>
-    <origin xyz="-0.054025 0.0 0.14405" rpy="0 0 0"/>
+    <child link="camera_link"/>
+    <origin xyz="-0.115 0.01 0.179" rpy="0 0 0"/>
   </joint>
   <link name="camera_link">
@@ -174,10 +174,10 @@
       <origin xyz="0 0 0 " rpy="0 0 1.570796" />
       <geometry>
-        <mesh filename="package://dami2_description/meshes/sensors/kinect.dae" scale="0.001 0.001 0.001"/>
-      </geometry>
-      <material name="dark"/>
-    </visual>
-    <collision>
-      <origin xyz="0 0 0" rpy="0 0 0" />
+        <mesh filename="package://dami2_description/meshes/sensors/kinect.stl" scale="0.001 0.001 0.001"/>
+      </geometry>
+      <material name="dark"/>
+    </visual>
+    <collision>
+      <origin xyz="0 0 0.0225" rpy="0 0 0" />
       <geometry>
         <box size="0.07271 0.27794 0.0720"/>
@@ -185,11 +185,32 @@
     </collision>
   </link>
-  <joint name="camera_depth_joint" type="fixed">
-    <origin xyz="0 0.01235 0.0" rpy="0 0 0" />
-    <parent link="camera_link" />
+<joint name="camera_depth_joint" type="fixed">
+    <origin xyz="-0.050 0.0 0.0805" rpy="0 0 0" />
+    <parent link="base_link" />
     <child link="camera_depth_frame" />
   </joint>
-  <link name="camera_depth_frame"/>
-  <joint name="camera_depth_optical_joint" type="fixed">
+  <link name="camera_depth_frame">
+  <inertial>
+      <mass value="0.17" />
+      <origin xyz="0 0 0" />
+      <inertia ixx="0.001" ixy="0.0" ixz="0.0"
+               iyy="0.001" iyz="0.0"
+               izz="0.001" />
+    </inertial>
+    <visual>
+      <origin xyz="0 0 0 " rpy="0 0 0" />
+      <geometry>
+        <mesh filename="package://dami2_description/meshes/sensors/lidar.stl" scale="0.001 0.001 0.001"/>
+      </geometry>
+      <material name="dark"/>
+    </visual>
+    <collision>
+      <origin xyz="0 0 0.030" rpy="0 0 0" />
+      <geometry>
+        <box size="0.070 0.100 0.060"/>
+      </geometry>
+    </collision>
+  </link>
+<joint name="camera_depth_optical_joint" type="fixed">
     <origin xyz="0 0 0" rpy="-1.5707963268 0 -1.5707963268" />
     <parent link="camera_depth_frame" />

Commit message: robot rev2

File: dami2_description/urdf/dami2.gazebo.xacro (robot description, xacro)
@@ -129,3 +129,31 @@
     </sensor>
   </gazebo>
+  <gazebo reference="rplidar_link">
+    <material>Gazebo/FlatBlack</material>
+    <sensor type="ray" name="slamtec_rplidar_sensor">
+      <pose>0 0 0 0 0 0</pose>
+      <visualize>$(arg laser_visual)</visualize>
+      <update_rate>5</update_rate>
+      <ray>
+        <scan>
+          <horizontal>
+            <samples>360</samples>
+            <resolution>1</resolution>
+            <min_angle>0.0</min_angle>
+            <max_angle>6.28319</max_angle>
+          </horizontal>
+        </scan>
+        <range>
+          <min>0.120</min>
+          <max>3.5</max>
+          <resolution>0.015</resolution>
+        </range>
+        <noise>
+          <type>gaussian</type>
+          <mean>0.0</mean>
+          <stddev>0.01</stddev>
+        </noise>
+      </ray>
+    </sensor>
+  </gazebo>
 </robot>

File: dami2_description/urdf/dami2.urdf.xacro (robot description, xacro)
@@ -160,11 +160,6 @@
   <joint name="scan_joint" type="fixed">
     <parent link="base_link"/>
-<<<<<<< HEAD
     <child link="camera_link"/>
     <origin xyz="-0.115 0.01 0.179" rpy="0 0 0"/>
-=======
-    <child link="camer_scan"/>
-    <origin xyz="-0.054025 0.0 0.14405" rpy="0 0 0"/>
->>>>>>> 8a5ce0be434e64339d8b732d660b9734f95c948f
   </joint>
   <link name="camera_link">
@@ -193,7 +188,7 @@
     <origin xyz="-0.050 0.0 0.0805" rpy="0 0 0" />
     <parent link="base_link" />
-    <child link="camera_depth_frame" />
-  </joint>
-  <link name="camera_depth_frame">
+    <child link="rplidar_link" />
+  </joint>
+  <link name="rplidar_link">
   <inertial>
       <mass value="0.17" />
@@ -219,5 +214,5 @@
 <joint name="camera_depth_optical_joint" type="fixed">
     <origin xyz="0 0 0" rpy="-1.5707963268 0 -1.5707963268" />
-    <parent link="camera_depth_frame" />
+    <parent link="rplidar_link" />
     <child link="camera_depth_optical_frame" />
   </joint>

Commit message: robot rev3

File: dami2_description/urdf/dami2.gazebo.xacro (robot description, xacro)
@@ -101,7 +101,7 @@
     </plugin>
   </gazebo>
-  <gazebo reference="camera_link">
+  <gazebo reference="depth_camera_link">
     <material>Gazebo/FlatBlack</material>
-    <sensor type="ray" name="lds_lfcd_sensor">
+    <sensor type="ray" name="kinect_sensor">
       <pose>0 0 0 0 0 0</pose>
       <visualize>$(arg laser_visual)</visualize>
@@ -131,21 +131,21 @@
   <gazebo reference="rplidar_link">
     <material>Gazebo/FlatBlack</material>
-    <sensor type="ray" name="slamtec_rplidar_sensor">
+    <sensor type="gpu_ray" name="slamtec_rplidar_sensor">
       <pose>0 0 0 0 0 0</pose>
       <visualize>$(arg laser_visual)</visualize>
-      <update_rate>5</update_rate>
+      <update_rate>10</update_rate>
       <ray>
         <scan>
           <horizontal>
-            <samples>360</samples>
+            <samples>400</samples>
             <resolution>1</resolution>
-            <min_angle>0.0</min_angle>
-            <max_angle>6.28319</max_angle>
+            <min_angle>-3.14159</min_angle>
+            <max_angle>3.14159</max_angle>
           </horizontal>
         </scan>
         <range>
-          <min>0.120</min>
-          <max>3.5</max>
-          <resolution>0.015</resolution>
+          <min>0.15</min>
+          <max>6.0</max>
+          <resolution>0.01</resolution>
         </range>
         <noise>

File: dami2_description/urdf/dami2.urdf.xacro (robot description, xacro)
@@ -160,10 +160,10 @@
   <joint name="scan_joint" type="fixed">
     <parent link="base_link"/>
-    <child link="camera_link"/>
+    <child link="depth_camera_link"/>
     <origin xyz="-0.115 0.01 0.179" rpy="0 0 0"/>
   </joint>
-  <link name="camera_link">
-    <inertial>
-      <mass value="0.114" />
+  <link name="depth_camera_link">
+    <inertial>
+      <mass value="0.01" />
       <origin xyz="0 0 0" />
       <inertia ixx="0.001" ixy="0.0" ixz="0.0"
@@ -181,9 +181,9 @@
       <origin xyz="0 0 0.0225" rpy="0 0 0" />
       <geometry>
-        <box size="0.07271 0.27794 0.0720"/>
-      </geometry>
-    </collision>
-  </link>
-<joint name="camera_depth_joint" type="fixed">
+        <box size="0.073 0.276 0.072"/>
+      </geometry>
+    </collision>
+  </link>
+  <joint name="rplidar_joint" type="fixed">
     <origin xyz="-0.050 0.0 0.0805" rpy="0 0 0" />
     <parent link="base_link" />
@@ -194,7 +194,7 @@
       <mass value="0.17" />
       <origin xyz="0 0 0" />
-      <inertia ixx="0.001" ixy="0.0" ixz="0.0"
-               iyy="0.001" iyz="0.0"
-               izz="0.001" />
+      <inertia ixx="1e-6" ixy="0.0" ixz="0.0"
+               iyy="1e-6" iyz="0.0"
+               izz="1e-6" />
     </inertial>
     <visual>
@@ -220,5 +220,5 @@
   <joint name="camera_rgb_joint" type="fixed">
     <origin xyz="0 -0.01235 0.0" rpy="0 0 0" />
-    <parent link="camera_link" />
+    <parent link="depth_camera_link" />
     <child link="camera_rgb_frame" />
   </joint>
